File: PhantomDriver_ER150D.brd (EAGLE design)
At the start: 160 x 116 mm, 231 parts, among them CN1 DF11-4DP-2DSA, CN10 826646-4, CN11 826646-4, CN12 BNC_ANGLE, CN13 BNC_ANGLE, CN14 BNC_ANGLE, CN15 DF11-4DP-2DSA, CN16 PCS-XE50LFD, CN17 PCS-XE50LFD, CN18 PH-2X5S, CN19 PIN_HEADER_SOCKET_14PIN, CN2 DF11-4DP-2DSA, CN20 DF11-14DP-2DSA, CN3 DF11-4DP-2DSA, CN4 DF11-4DP-2DSA, CN5 DF11-4DP-2DSA, CN6 DF11-4DP-2DSA, CN7 DF11-14DP-2DSA, CN8 PH-2X4S, CN9 DF11-4DP-2DSA, M1 VAB-3-10, M2 VAB-3-10, M3 VAB-3-10, SW1 A-12AV, SW2 A-12AV, SW3 A-12AV, SW4 A-12AV, U1 OPA2344EA, U10 74VHC4052AFT, U11 AD8227ARZ, U12 MAX4617CUE+, U13 MAX4617CUE+, U14 MAX4617CUE+, U15 MAX4617CUE+, U16 MAX4617CUE+, U17 MAX4617CUE+, U18 MAX4617CUE+, U19 MAX4617CUE+, U2 OPA2344EA, U20 MAX4617CUE+, U21 MAX4617CUE+, U22 MAX4617CUE+, U23 MAX4617CUE+, U24 MAX4617CUE+, U25 MAX4617CUE+, U26 TPS79933DDC, U27 5M160ZT100, U28 TPS79918DDC, U29 74VHC9541FT, U3 TS5A23159DGS, U30 TLP291GR, U4 TPS79933DDC, U5 OPA2344EA, U6 TPS3808G01DBV, U7 NJU7108F3, U8 OPA2344EA, U9 TS5A23159DGS

Commit message: 不具合修正完了
Parts:
- C1, C2, C6: value 47n -> 22n
- R12: value 50k/POT -> 20k/POT
- R3: value 270k -> 82k
- R5: value 43k -> 7.5k
- R6: value 330k -> 91k
- R7: value 270k -> 68k
- moved R59 21.2 mm to (9.14, 110.7), turned to 90 degrees
- moved R60 16.3 mm to (-11.2, 105.7), turned to 180 degrees
- moved D4 12.0 mm to (3.00, 111.0)
- moved D5 12.0 mm to (-9.00, 111.0)
- moved C58 5.08 mm to (7.11, 66.0)
- moved C59 5.08 mm to (7.11, 64.0)
- moved C60 5.08 mm to (7.11, 62.0)
- moved C61 5.08 mm to (7.11, 59.9)
- moved C62 5.08 mm to (7.11, 57.9)
- moved R72 5.08 mm to (2.03, 66.0)
- moved R73 5.08 mm to (2.03, 64.0)
- moved R74 5.08 mm to (2.03, 62.0)
- moved R75 5.08 mm to (2.03, 59.9)
- moved R76 5.08 mm to (2.03, 57.9)
Routing:
- net N$92: track 0.00 -> 36.0 mm, vias 0 -> 2
- net N$1: track 24.8 -> 37.4 mm, vias 0 -> 1
- net UI_VD+3V3: track 135.3 -> 126.9 mm
- net SW_!TEST!: track 4.53 -> 10.6 mm
- net SW_X1/!X2!: track 5.91 -> 11.8 mm
- net SW_INT/!EXT: track 9.94 -> 15.9 mm
- net SW_DDS/!ANALOG!: track 8.97 -> 14.9 mm
- net SW_X1/!X10!: track 7.37 -> 13.3 mm
- net VD+3V3: track 89.5 -> 85.9 mm
- net N$90: track 8.15 -> 5.51 mm
- net SW5: track 45.8 -> 46.9 mm
- net SW3: track 36.1 -> 37.2 mm
- net SW1: track 42.7 -> 43.7 mm
- net SW2: track 39.6 -> 40.6 mm
- net SW4: track 33.9 -> 34.9 mm
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Other:
- board text added: "2021/04"
- board text added: "Coil Driver 50ch"
- board text added: "CoilDriver 50ch UI"
- board text added: "DR20000193-00"
- board text added: "Eagle Tech."
- board text added: "EagleTech."
- board text removed: "2020/06"
- board text removed: "50ch Phantom Driver 3"
- board text removed: "50ch Phantom Driver3 UI"
- board text removed: "DR20000189-00"
- board text removed: "KIT Applied Electronics Lab."
- board text removed: "KIT/Applied Electronics Lab."
