File: 509_CoilDriver.brd (EAGLE design)
At the start: 160 x 116 mm, 231 parts, among them CN1 DF11-4DP-2DSA, CN10 826646-4, CN11 826646-4, CN12 BNC_ANGLE, CN13 BNC_ANGLE, CN14 BNC_ANGLE, CN15 DF11-4DP-2DSA, CN16 PCS-XE50LFD, CN17 PCS-XE50LFD, CN18 PH-2X5S, CN19 PIN_HEADER_SOCKET_14PIN, CN2 DF11-4DP-2DSA, CN20 DF11-14DP-2DSA, CN3 DF11-4DP-2DSA, CN4 DF11-4DP-2DSA, CN5 DF11-4DP-2DSA, CN6 DF11-4DP-2DSA, CN7 DF11-14DP-2DSA, CN8 PH-2X4S, CN9 DF11-4DP-2DSA, M1 VAB-3-10, M2 VAB-3-10, M3 VAB-3-10, SW1 A-12AV, SW2 A-12AV, SW3 A-12AV, SW4 A-12AV, U1 OPA2344EA, U10 74VHC4052AFT, U11 AD8227ARZ, U12 MAX4617CUE+, U13 MAX4617CUE+, U14 MAX4617CUE+, U15 MAX4617CUE+, U16 MAX4617CUE+, U17 MAX4617CUE+, U18 MAX4617CUE+, U19 MAX4617CUE+, U2 OPA2344EA, U20 MAX4617CUE+, U21 MAX4617CUE+, U22 MAX4617CUE+, U23 MAX4617CUE+, U24 MAX4617CUE+, U25 MAX4617CUE+, U26 TPS79933DDC, U27 5M160ZT100, U28 TPS79918DDC, U29 74VHC9541FT, U3 TS5A23159DGS, U30 TLP291GR, U4 TPS79933DDC, U5 OPA2344EA, U6 TPS3808G01DBV, U7 NJU7108F3, U8 OPA2344EA, U9 TS5A23159DGS

Commit message: modify Zout and Output Op-amps
Parts:
- R47, R51: value 100k -> 2.2k
- R48, R52: value 100k -> 22k
- R49: value 5.6k -> 200
- R50: value 39k -> 3.6k
- R53: value 10k -> 200
- R54: value 10k -> 39k
- R55: value 2k/0.05%/10ppm -> 82k/0.05%/10ppm
- R56: value 100/0.05%/10ppm -> 10/0.5%/5ppm
- R57: value 15k/0.05%/10ppm -> 20k/0.05%/10ppm
- U8: value OPA2344EA -> OPA2314AIDGK
Changed lines of the file:
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@@
 <attribute name="VALUE" x="108.331" y="62.865" size="1.016" layer="27" font="vector" ratio="12" rot="R270"/>
 </element>
-<element name="U8" library="AEL_linear" package="MSO8_AEL" value="OPA2344EA" x="123.952" y="58.928" smashed="yes" rot="R180">
+<element name="U8" library="AEL_linear" package="MSO8_AEL" value="OPA2314AIDGK" x="123.952" y="58.928" smashed="yes" rot="R180">
 <attribute name="NAME" x="120.777" y="59.055" size="1.016" layer="25" font="vector" ratio="12" rot="R270"/>
 <attribute name="VALUE" x="119.507" y="60.833" size="1.016" layer="27" font="vector" ratio="12" rot="R270"/>
@@
 <attribute name="VALUE" x="125.857" y="54.102" size="1.016" layer="27" font="vector" ratio="15" rot="R180"/>
 </element>
-<element name="R52" library="AEL_RLC" package="RM1608" value="100k" x="131.064" y="70.104" smashed="yes">
+<element name="R52" library="AEL_RLC" package="RM1608" value="22k" x="131.064" y="70.104" smashed="yes">
 <attribute name="NAME" x="133.223" y="69.596" size="1.016" layer="25" font="vector" ratio="15"/>
 <attribute name="VALUE" x="128.524" y="67.564" size="1.016" layer="27" font="vector" ratio="15"/>
 </element>
-<element name="R53" library="AEL_RLC" package="RM1608" value="10k" x="129.032" y="78.232" smashed="yes">
+<element name="R53" library="AEL_RLC" package="RM1608" value="200" x="129.032" y="78.232" smashed="yes">
 <attribute name="NAME" x="131.318" y="77.851" size="1.016" layer="25" font="vector" ratio="15"/>
 <attribute name="VALUE" x="126.492" y="75.692" size="1.016" layer="27" font="vector" ratio="15"/>
 </element>
-<element name="R48" library="AEL_RLC" package="RM1608" value="100k" x="131.064" y="64.008" smashed="yes">
+<element name="R48" library="AEL_RLC" package="RM1608" value="22k" x="131.064" y="64.008" smashed="yes">
 <attribute name="NAME" x="133.223" y="63.5" size="1.016" layer="25" font="vector" ratio="15"/>
 <attribute name="VALUE" x="128.524" y="61.468" size="1.016" layer="27" font="vector" ratio="15"/>
 </element>
-<element name="R49" library="AEL_RLC" package="RM1608" value="5.6k" x="129.032" y="72.136" smashed="yes">
+<element name="R49" library="AEL_RLC" package="RM1608" value="200" x="129.032" y="72.136" smashed="yes">
 <attribute name="NAME" x="131.318" y="71.628" size="1.016" layer="25" font="vector" ratio="15"/>
 <attribute name="VALUE" x="126.492" y="69.596" size="1.016" layer="27" font="vector" ratio="15"/>
@@
 <attribute name="VALUE" x="13.081" y="26.797" size="1.016" layer="27" font="vector" ratio="15" rot="R180"/>
 </element>
-<element name="R56" library="AEL_RLC" package="RM1608" value="100/0.05%/10ppm" x="137.795" y="53.213" smashed="yes" rot="R270">
+<element name="R56" library="AEL_RLC" package="RM1608" value="10/0.5%/5ppm" x="137.795" y="53.213" smashed="yes" rot="R270">
 <attribute name="NAME" x="139.827" y="52.578" size="1.016" layer="25" font="vector" ratio="15" rot="R90"/>
 <attribute name="VALUE" x="135.255" y="55.753" size="1.016" layer="27" font="vector" ratio="15" rot="R270"/>
@@
 <attribute name="LF-CMRR" value="90" x="133.096" y="50.8" size="1.778" layer="27" rot="R180" display="off"/>
 </element>
-<element name="R57" library="AEL_RLC" package="RM1608" value="15k/0.05%/10ppm" x="133.096" y="58.928" smashed="yes">
+<element name="R57" library="AEL_RLC" package="RM1608" value="20k/0.05%/10ppm" x="133.096" y="58.928" smashed="yes">
 <attribute name="NAME" x="131.826" y="60.071" size="1.016" layer="25" font="vector" ratio="15"/>
 <attribute name="VALUE" x="130.556" y="56.388" size="1.016" layer="27" font="vector" ratio="15"/>
 </element>
-<element name="R55" library="AEL_RLC" package="RM1608" value="2k/0.05%/10ppm" x="133.096" y="56.896" smashed="yes">
+<element name="R55" library="AEL_RLC" package="RM1608" value="82k/0.05%/10ppm" x="133.096" y="56.896" smashed="yes">
 <attribute name="NAME" x="135.128" y="56.388" size="1.016" layer="25" font="vector" ratio="15"/>
 <attribute name="VALUE" x="130.556" y="54.356" size="1.016" layer="27" font="vector" ratio="15"/>
@@
 <attribute name="VALUE" x="137" y="118.5" size="1.27" layer="27" font="vector" ratio="12"/>
 </element>
-<element name="R51" library="AEL_RLC" package="RM1608" value="100k" x="131.064" y="68.072" smashed="yes">
+<element name="R51" library="AEL_RLC" package="RM1608" value="2.2k" x="131.064" y="68.072" smashed="yes">
 <attribute name="NAME" x="133.223" y="67.564" size="1.016" layer="25" font="vector" ratio="15"/>
 <attribute name="VALUE" x="128.524" y="65.532" size="1.016" layer="27" font="vector" ratio="15"/>
 </element>
-<element name="R54" library="AEL_RLC" package="RM1608" value="10k" x="129.032" y="76.2" smashed="yes">
+<element name="R54" library="AEL_RLC" package="RM1608" value="39k" x="129.032" y="76.2" smashed="yes">
 <attribute name="NAME" x="131.318" y="75.692" size="1.016" layer="25" font="vector" ratio="15"/>
 <attribute name="VALUE" x="126.492" y="73.66" size="1.016" layer="27" font="vector" ratio="15"/>
 </element>
-<element name="R47" library="AEL_RLC" package="RM1608" value="100k" x="131.064" y="66.04" smashed="yes">
+<element name="R47" library="AEL_RLC" package="RM1608" value="2.2k" x="131.064" y="66.04" smashed="yes">
 <attribute name="NAME" x="133.223" y="65.532" size="1.016" layer="25" font="vector" ratio="15"/>
 <attribute name="VALUE" x="128.524" y="63.5" size="1.016" layer="27" font="vector" ratio="15"/>
 </element>
-<element name="R50" library="AEL_RLC" package="RM1608" value="39k" x="129.032" y="74.168" smashed="yes">
+<element name="R50" library="AEL_RLC" package="RM1608" value="3.6k" x="129.032" y="74.168" smashed="yes">
 <attribute name="NAME" x="131.191" y="73.787" size="1.016" layer="25" font="vector" ratio="15"/>
 <attribute name="VALUE" x="126.492" y="71.628" size="1.016" layer="27" font="vector" ratio="15"/>
